File: MP3 Player Simplified/Simple MP3 Player/Simple MP3 Player.kicad_sch (KiCad schematic)
At the start: 38 parts, among them J1 Conn_01x02_Pin, J2 Micro_SD_Card, J5 AudioJack3_SwitchTR, SW1 Power, SW2 SW_Wuerth_450301014042, SW3 Front keys center, SW4 front keys bottom, SW5 Front Keys right, SW6 front keys left, SW7 Front keys up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

Commit message: added notes for bodges
Other:
- note added: "IS 3v3 in. need to bodge wire here"
- note added: "Need to bodge pull all down to ground with 10k"
- note added: "need to bodge together"
Changed lines of the file:
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@@
 	(generator_version "9.0")
 	(paper "A4")
+	(text "need to bodge together"
+		(exclude_from_sim no)
+		(at 76.454 116.078 0)
+		(effects
+			(font
+				(size 1.27 1.27)
+			)
+		)
+	)
+	(text "IS 3v3 in. need to bodge wire here"
+		(exclude_from_sim no)
+		(at 284.226 98.044 0)
+		(effects
+			(font
+				(size 1.27 1.27)
+			)
+		)
+	)
+	(text "Need to bodge pull all down to ground with 10k"
+		(exclude_from_sim no)
+		(at 47.752 171.45 0)
+		(effects
+			(font
+				(size 1.27 1.27)
+			)
+		)
+	)
 	(junction
 		(at 58.42 50.8)
@@
 		)
 	)
+	(polyline
+		(pts
+			(xy 86.36 115.57) (xy 91.44 115.57)
+		)
+		(stroke
+			(width 0)
+			(type default)
+		)
+	)
 	(wire
 		(pts
@@
 		)
 	)
+	(polyline
+		(pts
+			(xy 63.5 172.72) (xy 72.39 172.72)
+		)
+		(stroke
+			(width 0)
+			(type default)
+		)
+	)
+	(polyline
+		(pts
+			(xy 257.81 97.79) (xy 266.7 97.79)
+		)
+		(stroke
+			(width 0)
+			(type default)
+		)
+	)
 	(wire
 		(pts
@@
 		)
 	)
+	(polyline
+		(pts
+			(xy 86.36 116.84) (xy 86.36 127)
+		)
+		(stroke
+			(width 0)
+			(type default)
+		)
+	)
 	(wire
 		(pts
@@
 		)
 	)
+	(polyline
+		(pts
+			(xy 72.39 153.67) (xy 72.39 172.72)
+		)
+		(stroke
+			(width 0)
+			(type default)
+		)
+	)
 	(wire
 		(pts
@@
 		)
 		(instances
-			(project ""
+			(project "Simple MP3 Player"
 				(path "/ccbb7322-c983-4293-9e85-784d7b3dc014"
 					(reference "SW8")
@@
 		)
 		(instances
-			(project ""
+			(project "Simple MP3 Player"
 				(path "/ccbb7322-c983-4293-9e85-784d7b3dc014"
 					(reference "R3")
@@
 		)
 		(instances
-			(project ""
+			(project "Simple MP3 Player"
 				(path "/ccbb7322-c983-4293-9e85-784d7b3dc014"
 					(reference "C1")
@@
 		)
 		(instances
-			(project ""
+			(project "Simple MP3 Player"
 				(path "/ccbb7322-c983-4293-9e85-784d7b3dc014"
 					(reference "TP1")
@@
 		)
 		(instances
-			(project ""
+			(project "Simple MP3 Player"
 				(path "/ccbb7322-c983-4293-9e85-784d7b3dc014"
 					(reference "#PWR06")
@@
 		)
 		(instances
-			(project ""
+			(project "Simple MP3 Player"
 				(path "/ccbb7322-c983-4293-9e85-784d7b3dc014"
 					(reference "SW2")
@@
 		)
 		(instances
-			(project ""
+			(project "Simple MP3 Player"
 				(path "/ccbb7322-c983-4293-9e85-784d7b3dc014"
 					(reference "U3")
@@
 		)
 		(instances
-			(project ""
+			(project "Simple MP3 Player"
 				(path "/ccbb7322-c983-4293-9e85-784d7b3dc014"
 					(reference "C7")
@@
 		)
 		(instances
-			(project ""
+			(project "Simple MP3 Player"
 				(path "/ccbb7322-c983-4293-9e85-784d7b3dc014"
 					(reference "U5")
@@
 		)
 		(instances
-			(project ""
+			(project "Simple MP3 Player"
 				(path "/ccbb7322-c983-4293-9e85-784d7b3dc014"
 					(reference "U1")
@@
 		)
 		(instances
-			(project ""
+			(project "Simple MP3 Player"
 				(path "/ccbb7322-c983-4293-9e85-784d7b3dc014"
 					(reference "SW3")
@@
 		)
 		(instances
-			(project ""
+			(project "Simple MP3 Player"
 				(path "/ccbb7322-c983-4293-9e85-784d7b3dc014"
 					(reference "J5")
@@
 		)
 		(instances
-			(project ""
+			(project "Simple MP3 Player"
 				(path "/ccbb7322-c983-4293-9e85-784d7b3dc014"
 					(reference "#PWR04")
@@
 		)
 		(instances
-			(project ""
+			(project "Simple MP3 Player"
 				(path "/ccbb7322-c983-4293-9e85-784d7b3dc014"
 					(reference "R6")
@@
 		)
 		(instances
-			(project ""
+			(project "Simple MP3 Player"
 				(path "/ccbb7322-c983-4293-9e85-784d7b3dc014"
 					(reference "#PWR03")
@@
 		)
 		(instances
-			(project ""
+			(project "Simple MP3 Player"
 				(path "/ccbb7322-c983-4293-9e85-784d7b3dc014"
 					(reference "SW7")
@@
 		)
 		(instances
-			(project ""
+			(project "Simple MP3 Player"
 				(path "/ccbb7322-c983-4293-9e85-784d7b3dc014"
 					(reference "#PWR02")
@@
 		)
 		(instances
-			(project ""
+			(project "Simple MP3 Player"
 				(path "/ccbb7322-c983-4293-9e85-784d7b3dc014"
 					(reference "#PWR07")
@@
 		)
 		(instances
-			(project ""
+			(project "Simple MP3 Player"
 				(path "/ccbb7322-c983-4293-9e85-784d7b3dc014"
 					(reference "J2")
@@
 		)
 		(instances
-			(project ""
+			(project "Simple MP3 Player"
 				(path "/ccbb7322-c983-4293-9e85-784d7b3dc014"
 					(reference "R2")
@@
 		)
 		(instances
-			(project ""
+			(project "Simple MP3 Player"
 				(path "/ccbb7322-c983-4293-9e85-784d7b3dc014"
 					(reference "#PWR01")
@@
 		)
 		(instances
-			(project ""
+			(project "Simple MP3 Player"
 				(path "/ccbb7322-c983-4293-9e85-784d7b3dc014"
 					(reference "#PWR05")
@@
 		)
 		(instances
-			(project ""
+			(project "Simple MP3 Player"
 				(path "/ccbb7322-c983-4293-9e85-784d7b3dc014"
 					(reference "J1")
@@
 		)
 		(instances
-			(project ""
+			(project "Simple MP3 Player"
 				(path "/ccbb7322-c983-4293-9e85-784d7b3dc014"
 					(reference "R1")
@@
 		)
 		(instances
-			(project ""
+			(project "Simple MP3 Player"
 				(path "/ccbb7322-c983-4293-9e85-784d7b3dc014"
 					(reference "U2")
@@
 		)
 		(instances
-			(project ""
+			(project "Simple MP3 Player"
 				(path "/ccbb7322-c983-4293-9e85-784d7b3dc014"
 					(reference "C4")
@@
 		)
 		(instances
-			(project ""
+			(project "Simple MP3 Player"
 				(path "/ccbb7322-c983-4293-9e85-784d7b3dc014"
 					(reference "C13")
@@
 		)
 		(instances
-			(project ""
+			(project "Simple MP3 Player"
 				(path "/ccbb7322-c983-4293-9e85-784d7b3dc014"
 					(reference "C2")
